File: 3x2-macropad.kicad_sch (KiCad schematic)
At the start: 0 parts

Commit message: Version 1
Parts:
- added JP1: Jumper_2_Open, TestPoint:TestPoint_2Pads_Pitch2.54mm_Drill0.8mm, symbol Jumper:Jumper_2_Open
- added SW1, SW2, SW3, SW4, SW5, SW6: MX, Keebio-Parts:MX-Alps-Choc-1U-NoLED, symbol keebio:MX
- added U1: ProMicro, Keebio-Parts:ArduinoProMicro-ZigZag, symbol keebio:ProMicro
Connections:
- new net: JP1.1 (A), U1.22 (RST)
- new net 1x1: SW1.1, U1.5 (2/PD1)
- new net 1x2: SW3.1, U1.6 (3/PD0)
- new net 1x3: SW5.1, U1.7 (4/PD4)
- new net 2x1: SW2.1, U1.20 (A3/PF4)
- new net 2x2: SW4.1, U1.19 (A2/PF5)
- new net 2x3: SW6.1, U1.18 (A1/PF6)
- new net GND: JP1.2 (B), SW1.2, SW2.2, SW3.2, SW4.2, SW5.2, SW6.2, U1.23 (GND), U1.3 (GND), U1.4 (GND)
- no-connect marks 0 -> 14
